Commit message: urdf corrected

File: 3DModel/urdf/unnamed.urdf (robot description, URDF)
Before this commit: robot unnamed, 8 links, 7 joints
Links:
- removed link Cylinder_link
- added link base_link
Joints:
- joint joint1: parent Cylinder_link -> base_link
- joint joint7: limit lower=1.00000 upper=0.00000 effort=0.00000 velocity=0.00000 -> lower=0.00000 upper=1.00000 effort=0.00000 velocity=0.00000; origin xyz=1.03191 -2.31173 0.00000 rpy=-1.57080 0.00000 3.14159 -> xyz=1.03191 -2.90919 0.00000 rpy=-1.57080 0.00000 3.14159
