Commit message: Update robot model scaling and orientation for new units
Adjusted joint translations and scaling in openSCADModel2.scad and unnamed.urdf to use larger units (factor of 20), updated camera and platform settings, and added import of test1.stl. Modified ikpyErosion.py to support target orientation vectors and updated function signatures accordingly. Added test1.stl to the project.

File: Python-prototype/unnamed.urdf (robot description, URDF)
Before this commit: robot unnamed, 8 links, 7 joints
Links:
- added link vertical_tool
Joints:
- added joint tool_attachment_joint: type fixed, parent Cylinder.001_link, child vertical_tool, origin xyz=0 0 0 rpy=0 0 0
- joint joint1: origin xyz=0.08128 -0.00000 0.10051 rpy=-0.00000 -0.00000 0.00000 -> xyz=16.256 -0.00000 20.102 rpy=-0.00000 -0.00000 0.00000
- joint joint2: origin xyz=0.00572 -0.00000 0.15834 rpy=1.57080 0.00000 0.00000 -> xyz=1.144 -0.00000 31.668 rpy=1.57080 0.00000 0.00000
- joint joint3: origin xyz=-0.07496 0.11978 -0.00004 rpy=0.00000 0.00000 0.00000 -> xyz=-14.992 23.956 -0.008 rpy=0.00000 0.00000 0.00000
- joint joint4: origin xyz=0.04896 0.10337 0.00004 rpy=0.00000 0.00000 0.00000 -> xyz=9.792 20.674 0.008 rpy=0.00000 0.00000 0.00000
- joint joint5: origin xyz=0.10886 0.00722 -0.00004 rpy=-1.57080 0.00000 -1.57080 -> xyz=21.772 1.444 -0.008 rpy=-1.57080 0.00000 -1.57080
- joint joint6: origin xyz=0.00129 -0.00004 0.11812 rpy=1.57080 -1.57080 0.00000 -> xyz=0.258 -0.008 23.624 rpy=1.57080 -1.57080 0.00000
- joint joint7: limit lower=0.00000 upper=0.10000 effort=0.00000 velocity=0.00000 -> lower=0.00000 upper=20.00000 effort=0.00000 velocity=0.00000; origin xyz=0.10319 -0.29092 0.00000 rpy=-1.57080 0.00000 3.14159 -> xyz=20.638 -58.184 0.00000 rpy=-1.57080 0.00000 3.14159

Commit message: Update manipulator config, scale, and add main interface
Updated all manipulator configuration files (config.scad, openSCADModel2.scad, unnamed.urdf) to use new, larger scale and positions. Refactored ikpyErosion.py to improve interface and configuration generation, removing unused code. Added main.py to parse G-code and generate manipulator configurations layer by layer. Updated test.py to use the new G-code file. Added /Python-prototype/imgs to .gitignore.

File: Python-prototype/unnamed.urdf (robot description, URDF)
Before this commit: robot unnamed, 9 links, 8 joints
Joints:
- joint joint1: origin xyz=16.256 -0.00000 20.102 rpy=-0.00000 -0.00000 0.00000 -> xyz=81.280 0.00000 100.510 rpy=-0.00000 -0.00000 0.00000
- joint joint2: origin xyz=1.144 -0.00000 31.668 rpy=1.57080 0.00000 0.00000 -> xyz=5.720 0.00000 158.340 rpy=1.57080 0.00000 0.00000
- joint joint3: origin xyz=-14.992 23.956 -0.008 rpy=0.00000 0.00000 0.00000 -> xyz=-74.960 119.780 -0.040 rpy=0.00000 0.00000 0.00000
- joint joint4: origin xyz=9.792 20.674 0.008 rpy=0.00000 0.00000 0.00000 -> xyz=48.960 103.370 0.040 rpy=0.00000 0.00000 0.00000
- joint joint5: origin xyz=21.772 1.444 -0.008 rpy=-1.57080 0.00000 -1.57080 -> xyz=108.860 7.220 -0.040 rpy=-1.57080 0.00000 -1.57080
- joint joint6: origin xyz=0.258 -0.008 23.624 rpy=1.57080 -1.57080 0.00000 -> xyz=1.290 -0.040 118.120 rpy=1.57080 -1.57080 0.00000
- joint joint7: limit lower=0.00000 upper=20.00000 effort=0.00000 velocity=0.00000 -> lower=0.00000 upper=100.00000 effort=0.00000 velocity=0.00000; origin xyz=20.638 -58.184 0.00000 rpy=-1.57080 0.00000 3.14159 -> xyz=103.190 -290.920 0.00000 rpy=-1.57080 0.00000 3.14159
